File: board/fancontroller.sch (EAGLE design)
At the start: 3 parts

Commit message: Capturing protoboard layout
Parts:
- removed U$2: ATTINY13DIP, SparkFun-DigitalIC:ATTINY13DIP
- added C10: 1uF, SparkFun-Capacitors:CAPPTH
- added C2, C3, C4, C5, C6: 0.1uF, SparkFun-Capacitors:CAPPTH
- added C7: 100uF, SparkFun-Capacitors:CAP_POLPTH1
- added C8: 1000uF, SparkFun-Capacitors:CAP_POLPTH1
- added C9: 10uF, SparkFun-Capacitors:CAPPTH
- added D1: 1N5818-B, diode:1N5818-B
- added D2: Yellow, SparkFun-LED:LED5MM
- added D3: 5.5V, SparkFun-DiscreteSemi:DIODE-ZENERPTH
- added IC1: AVR-MEGA168-PTH, SparkFun-DigitalIC:AVR-MEGA8-PPTH
- added IC3: LM7805, linear:7812TV
- added IC4: LM358, SparkFun-AnalogIC:LM358KIT
- added J1: AVR_SPI_PRG_6OFFSET_PADS, SparkFun-Connectors:AVR_SPI_PRG_6OFFSET_PADS
- added L1: 100uH, inductors:A26GFC
- added R1: 10k, SparkFun-Resistors:10KOHM-1/4W-1%(PTH)VERT
- added R2: 100k, SparkFun-Resistors:10KOHM-1/4W-1%(PTH)VERT
- added R3: 33k, SparkFun-Resistors:10KOHM-1/4W-1%(PTH)VERT
- added R4: 11k, SparkFun-Resistors:10KOHM-1/4W-1%(PTH)VERT
- added R5: 1k, SparkFun-Resistors:10KOHM-1/4W-1%(PTH)VERT
- added R6: 150, SparkFun-Resistors:10KOHM-1/4W-1%(PTH)VERT
- added R7: 100, SparkFun-Resistors:10KOHM-1/4W-1%(PTH)VERT
- added R8: 10k, SparkFun-Electromechanical:TRIMPOTPTH
- added U1: TMP35, SparkFun-Sensors:TMP36GT9
- U$3: value MCP41X1 -> MCP4131-103
Connections:
- new net /RESET: IC1.PC6(/RESET), J1.5, R5.1
- new net /SS: IC1.PB2(SS/OC1B), U$3./CS
- new net 12V: C7.+, C9.1, IC3.VI, IC4G1.V+, U$1.VIN
- new net 5V: C10.1, C2.1, C4.1, IC1.VCC@1, IC3.VO, J1.2, R5.2, R6.1, U$3.P0B, U$3.VDD, U1.VCC
- new net GND: C10.2, C2.2, C3.2, C4.2, C5.2, C6.2, C7.-, C8.-, C9.2, D1.A, D3.A, IC1.AGND, IC1.GND@1, IC3.GND, IC4G1.V-, J1.6, R4.1, R7.1, R8.CCW, U$1./ON, U$1.GND, U$3.P0A, U$3.VSS, U1.GND
- new net MISO: IC1.PB4(MISO), J1.1
- new net MOSI: IC1.PB3(MOSI/OC2), J1.4, U$3.SDI/SDO
- new net N$1: C8.+, L1.2, R8.CW
- new net N$11: C3.1, R1.1, U1.VOUT
- new net N$2: D2.A, IC1.PB0(ICP)
- new net N$3: D1.C, L1.1, U$1.OUTPUT
- new net N$4: R8.WIPER, U$1.FEEDBACK
- new net N$5: D2.C, R7.2
- new net N$6: IC4G1.OUT, R2.1, R3.2
- new net N$7: IC4G1.-IN, R3.1, R4.2
- new net N$8: IC4G1.+IN, R1.2
- new net N$9: C6.1, IC1.AREF, R6.2
- new net POT_P0W: U$3.P0W
- new net SCK: IC1.PB5(SCK), J1.3, U$3.SCK
- new net TEMP_SENSOR: C5.1, D3.C, IC1.PC0(ADC0), R2.2
Other:
- note added: "/RESET"
- note added: "Av = 4"
- note added: "FAN+"
- note added: "FAN-"
- note added: "Notes: - Temp sensor output can damage uC - Digital pot needs to go through op-amp to scale feedback voltage - DC/DC converter feedback needs to incorporate temp sensor"
- note added: "TMP35: - 25°C = 250mV - 10°C to 125°C - 100mV to 1250mV - 10mV/°C - Transfer function: F(x) = 1/100x"
- note added: "Temp Sensor"
- note added: "Temp Sensor Scaled Output: - 400mV to 5000mV"
